Commit message: mod: remove Gazebo material overrides from robot models
Signed-off-by: Tomoaki Fujino <fujino.tomoaki404@mail.kyutech.jp>

File: turtlebot3_lime_gazebo/urdf/open_manipulator_sara.gazebo.xacro (robot description, xacro)
@@ -2,9 +2,5 @@
 <robot xmlns:xacro="http://www.ros.org/wiki/xacro">
   <xacro:macro name="open_manipulator_sara_gazebo" params="prefix">
-    <xacro:macro name="Link" params="reference">
-      <gazebo reference="${reference}">
-        <material>Gazebo/DarkGrey</material>
-      </gazebo>
-    </xacro:macro>
+    <xacro:macro name="Link" params="reference"/>
     <xacro:Link reference="${prefix}link1"/>
     <xacro:Link reference="${prefix}link2"/>
@@ -16,16 +12,4 @@
     <xacro:Link reference="${prefix}gripper_left_link"/>
     <xacro:Link reference="${prefix}gripper_right_link"/>
-    <gazebo reference="${prefix}link1">
-      <material>Gazebo/Green</material>
-    </gazebo>
-    <gazebo reference="${prefix}link3">
-      <material>Gazebo/Green</material>
-    </gazebo>
-    <gazebo reference="${prefix}link5">
-      <material>Gazebo/Green</material>
-    </gazebo>
-    <gazebo reference="${prefix}end_effector_link">
-      <material>Gazebo/Red</material>
-    </gazebo>
   </xacro:macro>
 </robot>

File: turtlebot3_lime_gazebo/urdf/sensors/imu.gazebo.xacro (robot description, xacro)
@@ -5,5 +5,4 @@
     params="prefix">
     <gazebo reference="${prefix}imu_link">
-      <material>Gazebo/Grey</material>
       <sensor name="imu" type="imu">
         <always_on>true</always_on>

File: turtlebot3_lime_gazebo/urdf/sensors/lidar.gazebo.xacro (robot description, xacro)
@@ -5,5 +5,4 @@
     params="prefix">
     <gazebo reference="${prefix}base_scan">
-      <material>Gazebo/FlatBlack</material>
       <sensor name="lidar" type="gpu_lidar">
         <pose>0 0 0 0 0 0</pose>

File: turtlebot3_lime_gazebo/urdf/turtlebot3_bigwheel_orin.gazebo.xacro (robot description, xacro)
@@ -8,34 +8,19 @@
     filename="$(find turtlebot3_lime_gazebo)/urdf/sensors/rgbd_camera.gazebo.xacro" />
   <xacro:macro name="turtlebot3_bigwheel_orin_gazebo" params="prefix">
-    <gazebo reference="${prefix}base_link">
-      <material>Gazebo/DarkGrey</material>
-    </gazebo>
     <gazebo reference="${prefix}wheel_left_link">
       <mu1>1.0</mu1>
       <mu2>1.0</mu2>
-      <material>
-        <ambient>0.0 0.8 0.0 1.0</ambient>
-        <diffuse>0.0 0.8 0.0 1.0</diffuse>
-        <specular>0.1 0.1 0.1 1.0</specular>
-      </material>
     </gazebo>
     <gazebo reference="${prefix}wheel_right_link">
       <mu1>1.0</mu1>
       <mu2>1.0</mu2>
-      <material>
-        <ambient>0.0 0.8 0.0 1.0</ambient>
-        <diffuse>0.0 0.8 0.0 1.0</diffuse>
-        <specular>0.1 0.1 0.1 1.0</specular>
-      </material>
     </gazebo>
     <gazebo reference="${prefix}caster_back_right_link">
       <mu1>0.1</mu1>
       <mu2>0.1</mu2>
-      <material>Gazebo/FlatBlack</material>
     </gazebo>
     <gazebo reference="${prefix}caster_back_left_link">
       <mu1>0.1</mu1>
       <mu2>0.1</mu2>
-      <material>Gazebo/FlatBlack</material>
     </gazebo>
     <xacro:turtlebot3_lime_imu_gazebo
