Commit message: new: migrate simulation to Gazebo Sim in a dedicated package
Signed-off-by: Tomoaki Fujino <fujino.tomoaki404@mail.kyutech.jp>

File: turtlebot3_lime_description/urdf/open_manipulator_sara.urdf.xacro (robot description, xacro)
@@ -6,5 +6,5 @@
 -->
 <robot xmlns:xacro="http://www.ros.org/wiki/xacro">
-  <xacro:macro name="open_manipulator_sara" params="prefix">
+  <xacro:macro name="open_manipulator_sara" params="prefix arm_friction:=1.0 gripper_friction:=1.0">
     <xacro:property name="meshes_file_direction" value="package://turtlebot3_lime_description/meshes/open_manipulator_sara"/>
     <link name="${prefix}link1">
@@ -14,5 +14,5 @@
           <mesh filename="${meshes_file_direction}/link1.stl" scale="0.001 0.001 0.001"/>
         </geometry>
-        <material name="grey"/>
+        <material name="black"/>
       </visual>
       <collision>
@@ -34,5 +34,5 @@
       <axis xyz="0 0 1"/>
       <limit velocity="4.8" effort="1" lower="${-pi*0.9}" upper="${pi*0.9}" />
-      <dynamics damping="0.7" friction="1.0"/>
+      <dynamics damping="0.7" friction="${arm_friction}"/>
     </joint>
     <link name="${prefix}link2">
@@ -42,5 +42,5 @@
           <mesh filename="${meshes_file_direction}/link2.stl" scale="0.001 0.001 0.001"/>
         </geometry>
-        <material name="grey"/>
+        <material name="green"/>
       </visual>
       <collision>
@@ -62,5 +62,5 @@
       <axis xyz="0 1 0"/>
       <limit velocity="4.8" effort="1" lower="${-pi*0.541}" upper="${pi*0.562}" />
-      <dynamics damping="0.7" friction="1.0"/>
+      <dynamics damping="0.7" friction="${arm_friction}"/>
     </joint>
     <link name="${prefix}link3">
@@ -70,5 +70,5 @@
           <mesh filename="${meshes_file_direction}/link3.stl" scale="0.001 0.001 0.001"/>
         </geometry>
-        <material name="grey"/>
+        <material name="black"/>
       </visual>
       <collision>
@@ -90,5 +90,5 @@
       <axis xyz="0 1 0"/>
       <limit velocity="4.8" effort="1" lower="${-pi*0.560}" upper="${pi*0.591}" />
-      <dynamics damping="0.7" friction="1.0"/>
+      <dynamics damping="0.7" friction="${arm_friction}"/>
     </joint>
     <link name="${prefix}link4">
@@ -98,5 +98,5 @@
           <mesh filename="${meshes_file_direction}/link4.stl" scale="0.001 0.001 0.001"/>
         </geometry>
-        <material name="grey"/>
+        <material name="green"/>
       </visual>
       <collision>
@@ -118,5 +118,5 @@
       <axis xyz="0 0 1"/>
       <limit velocity="4.8" effort="1" lower="${-pi*0.5}" upper="${pi*0.5}" />
-      <dynamics damping="0.7" friction="1.0"/>
+      <dynamics damping="0.7" friction="${arm_friction}"/>
     </joint>
     <link name="${prefix}link5">
@@ -126,5 +126,5 @@
           <mesh filename="${meshes_file_direction}/link5.stl" scale="0.001 0.001 0.001"/>
         </geometry>
-        <material name="grey"/>
+        <material name="black"/>
       </visual>
       <collision>
@@ -146,5 +146,5 @@
       <axis xyz="0 1 0"/>
       <limit velocity="4.8" effort="1" lower="${-pi*0.531}" upper="${pi*0.567}" />
-      <dynamics damping="0.7" friction="1.0"/>
+      <dynamics damping="0.7" friction="${arm_friction}"/>
     </joint>
     <link name="${prefix}link6">
@@ -154,5 +154,5 @@
           <mesh filename="${meshes_file_direction}/link6.stl" scale="0.001 0.001 0.001"/>
         </geometry>
-        <material name="grey"/>
+        <material name="green"/>
       </visual>
       <collision>
@@ -179,5 +179,5 @@
       <axis xyz="0 0 1"/>
       <limit velocity="4.8" effort="1" lower="${-pi*0.9}" upper="${pi*0.9}" />
-      <dynamics damping="0.7" friction="1.0"/>
+      <dynamics damping="0.7" friction="${arm_friction}"/>
     </joint>
     <link name="${prefix}link7">
@@ -187,5 +187,5 @@
           <mesh filename="${meshes_file_direction}/link7.stl" scale="0.001 0.001 0.001"/>
         </geometry>
-        <material name="grey"/>
+        <material name="black"/>
       </visual>
       <collision>
@@ -207,5 +207,5 @@
           <mesh filename="${meshes_file_direction}/gripper_left_palm.stl" scale="0.001 0.001 0.001"/>
         </geometry>
-        <material name="grey"/>
+        <material name="black"/>
       </visual>
       <collision>
@@ -227,5 +227,5 @@
       <axis xyz="0 1 0"/>
       <limit velocity="4.8" effort="1" lower="-0.010" upper="0.019" />
-      <dynamics damping="0.7" friction="1.0"/>
+      <dynamics damping="0.7" friction="${gripper_friction}"/>
     </joint>
     <!-- Move it 2 not find mimic-->
@@ -243,5 +243,5 @@
       <limit velocity="4.8" effort="1" lower="-0.010" upper="0.019" />
       <mimic joint="${prefix}gripper_left_joint" multiplier="1"/>
-      <dynamics damping="0.7" friction="1.0"/>
+      <dynamics damping="0.7" friction="${gripper_friction}"/>
     </joint>
     <link name="${prefix}gripper_right_link">
@@ -251,5 +251,5 @@
           <mesh filename="${meshes_file_direction}/gripper_right_palm.stl" scale="0.001 0.001 0.001"/>
         </geometry>
-        <material name="grey"/>
+        <material name="black"/>
       </visual>
       <collision>
@@ -276,5 +276,5 @@
           <box size="0.01 0.01 0.01" />
         </geometry>
-        <material name="grey"/>
+        <material name="red"/>
       </visual>
       <inertial>

File: turtlebot3_lime_description/urdf/turtlebot3_bigwheel_orin.urdf.xacro (robot description, xacro)
@@ -21,5 +21,5 @@
           <mesh filename="${meshes_file_direction}/base.stl" scale="0.001 0.001 0.001"/>
         </geometry>
-        <material name="light_black"/>
+        <material name="black"/>
       </visual>
       <collision>
@@ -50,5 +50,5 @@
           <mesh filename="${meshes_file_direction}/tire.stl" scale="0.001 0.001 0.001"/>
         </geometry>
-        <material name="dark"/>
+        <material name="green"/>
       </visual>
       <collision>
@@ -78,5 +78,5 @@
           <mesh filename="${meshes_file_direction}/tire.stl" scale="0.001 0.001 0.001"/>
         </geometry>
-        <material name="dark"/>
+        <material name="green"/>
       </visual>
       <collision>
@@ -107,5 +107,5 @@
           <sphere radius="0.005"/>
         </geometry>
-        <material name="dark"/>
+        <material name="black"/>
       </visual>
       <inertial>
@@ -130,5 +130,5 @@
           <sphere radius="0.005"/>
         </geometry>
-        <material name="dark"/>
+        <material name="black"/>
       </visual>
       <inertial>
@@ -155,5 +155,5 @@
           <mesh filename="${meshes_file_direction}/ladar.stl" scale="0.001 0.001 0.001"/>
         </geometry>
-        <material name="dark"/>
+        <material name="black"/>
       </visual>
       <collision>

File: turtlebot3_lime_description/urdf/turtlebot3_lime.urdf.xacro (robot description, xacro)
@@ -4,22 +4,17 @@
   xmlns:xacro="http://www.ros.org/wiki/xacro">
   <xacro:arg name="prefix" default="" />
-  <xacro:arg name="use_sim" default="false" />
+  <xacro:arg name="use_gazebo" default="false" />
   <xacro:arg name="use_fake_hardware" default="false" />
   <xacro:arg name="fake_sensor_commands" default="false" />
   <!-- Import materials macro -->
-  <xacro:include filename="$(find turtlebot3_lime_description)/gazebo/materials.xacro" />
-  <!-- Include TurtleBot3 Waffle Pi urdf macro -->
+  <xacro:include filename="$(find turtlebot3_lime_description)/urdf/materials.urdf.xacro" />
+  <!-- Include TurtleBot3 BigWheel Orin URDF macro -->
   <xacro:include filename="$(find turtlebot3_lime_description)/urdf/turtlebot3_bigwheel_orin.urdf.xacro" />
-  <!-- Include TurtleBot3 Waffle Pi gazebo macro -->
-  <xacro:include filename="$(find turtlebot3_lime_description)/gazebo/turtlebot3_bigwheel_orin.gazebo.xacro" />
   <!-- Include OpenManipulator-X urdf macro -->
   <xacro:include filename="$(find turtlebot3_lime_description)/urdf/open_manipulator_sara.urdf.xacro" />
-  <!-- Include OpenManipulator-X gazebo macro -->
-  <xacro:include filename="$(find turtlebot3_lime_description)/gazebo/open_manipulator_sara.gazebo.xacro" />
-  <!-- Include TurtleBot3 Lime ros2 control macro -->
-  <xacro:include filename="$(find turtlebot3_lime_description)/ros2_control/turtlebot3_lime_system.ros2_control.xacro" />
+  <!-- Include TurtleBot3 Lime System urdf macro -->
+  <xacro:include filename="$(find turtlebot3_lime_description)/urdf/control/turtlebot3_lime_system.ros2_control.xacro"/>
   <xacro:turtlebot3_bigwheel_orin prefix="$(arg prefix)" />
-  <xacro:turtlebot3_bigwheel_orin_gazebo prefix="$(arg prefix)" />
-  <!-- Used for fixing OpenManipulator-X on TurtleBot3 Waffle Pi -->
+  <!-- Fixed joint between the mobile base and manipulator -->
   <joint name="$(arg prefix)base_fixed" type="fixed">
     <parent link="$(arg prefix)base_link"/>
@@ -28,10 +23,9 @@
   </joint>
   <xacro:open_manipulator_sara prefix="$(arg prefix)" />
-  <xacro:open_manipulator_sara_gazebo prefix="$(arg prefix)" />
-  <xacro:turtlebot3_lime_system name="TurtleBot3LimeSystem" prefix="$(arg prefix)" use_sim="$(arg use_sim)" use_fake_hardware="$(arg use_fake_hardware)" fake_sensor_commands="$(arg fake_sensor_commands)"/>
-  <gazebo>
-    <plugin name="gazebo_ros2_control" filename="libgazebo_ros2_control.so">
-      <parameters>$(find turtlebot3_lime_bringup)/config/gazebo_controller_manager.yaml</parameters>
-    </plugin>
-  </gazebo>
+  <xacro:turtlebot3_lime_system
+    name="TurtleBot3LimeSystem"
+    prefix="$(arg prefix)"
+    use_gazebo="$(arg use_gazebo)"
+    use_fake_hardware="$(arg use_fake_hardware)"
+    fake_sensor_commands="$(arg fake_sensor_commands)"/>
 </robot>

Commit message: fix: omit gripper URDF mimic tag when using Gazebo
Signed-off-by: Tomoaki Fujino <fujino.tomoaki404@mail.kyutech.jp>

File: turtlebot3_lime_description/urdf/open_manipulator_sara.urdf.xacro (robot description, xacro)
@@ -6,5 +6,5 @@
 -->
 <robot xmlns:xacro="http://www.ros.org/wiki/xacro">
-  <xacro:macro name="open_manipulator_sara" params="prefix arm_friction:=1.0 gripper_friction:=1.0">
+  <xacro:macro name="open_manipulator_sara" params="prefix use_gazebo:=false arm_friction:=1.0 gripper_friction:=1.0">
     <xacro:property name="meshes_file_direction" value="package://turtlebot3_lime_description/meshes/open_manipulator_sara"/>
     <link name="${prefix}link1">
@@ -242,5 +242,7 @@
       <axis xyz="0 -1 0"/>
       <limit velocity="4.8" effort="1" lower="-0.010" upper="0.019" />
-      <mimic joint="${prefix}gripper_left_joint" multiplier="1"/>
+      <xacro:unless value="${use_gazebo}">
+        <mimic joint="${prefix}gripper_left_joint" multiplier="1"/>
+      </xacro:unless>
       <dynamics damping="0.7" friction="${gripper_friction}"/>
     </joint>

File: turtlebot3_lime_description/urdf/turtlebot3_lime.urdf.xacro (robot description, xacro)
@@ -22,5 +22,5 @@
     <origin xyz="-0.036 0.0 0.07" rpy="0 0 0"/>
   </joint>
-  <xacro:open_manipulator_sara prefix="$(arg prefix)" />
+  <xacro:open_manipulator_sara prefix="$(arg prefix)" use_gazebo="$(arg use_gazebo)" arm_friction="1.0" gripper_friction="1.0"/>
   <xacro:turtlebot3_lime_system
     name="TurtleBot3LimeSystem"

File: turtlebot3_lime_gazebo/urdf/turtlebot3_lime.urdf.xacro (robot description, xacro)
@@ -28,5 +28,5 @@
   </joint>
   <!-- Reduced simulation friction: effort limits are 1 N m (arm) and 1 N (gripper). -->
-  <xacro:open_manipulator_sara prefix="$(arg prefix)" arm_friction="0.01" gripper_friction="0.01" />
+  <xacro:open_manipulator_sara prefix="$(arg prefix)" use_gazebo="true" arm_friction="0.01" gripper_friction="0.01" />
   <xacro:turtlebot3_bigwheel_orin_gazebo prefix="$(arg prefix)" />
   <xacro:open_manipulator_sara_gazebo prefix="$(arg prefix)" />

Commit message: fix: restore gripper mimic joint in Gazebo URDF
Signed-off-by: Tomoaki Fujino <fujino.tomoaki404@mail.kyutech.jp>

File: turtlebot3_lime_description/urdf/open_manipulator_sara.urdf.xacro (robot description, xacro)
@@ -242,7 +242,5 @@
       <axis xyz="0 -1 0"/>
       <limit velocity="4.8" effort="1" lower="-0.010" upper="0.019" />
-      <xacro:unless value="${use_gazebo}">
-        <mimic joint="${prefix}gripper_left_joint" multiplier="1"/>
-      </xacro:unless>
+      <mimic joint="${prefix}gripper_left_joint" multiplier="1"/>
       <dynamics damping="0.7" friction="${gripper_friction}"/>
     </joint>
