Commit message: fix: support Jazzy teleop and Servo with continuous joint commands
Signed-off-by: Tomoaki Fujino <fujino.tomoaki404@mail.kyutech.jp>

File: turtlebot3_lime_description/urdf/control/turtlebot3_lime_system.ros2_control.xacro (robot description, xacro)
@@ -6,4 +6,5 @@
 -->
 <robot xmlns:xacro="http://www.ros.org/wiki/xacro">
+  <xacro:property name="ros_distro" value="$(env ROS_DISTRO)" />
   <xacro:macro
     name="turtlebot3_lime_system"
@@ -208,7 +209,14 @@
           </parameters>
           <ros>
-            <remapping>
-              /diff_drive_controller/cmd_vel_unstamped:=/cmd_vel
-            </remapping>
+            <xacro:if value="${ros_distro == 'humble'}">
+              <remapping>
+                /diff_drive_controller/cmd_vel_unstamped:=/cmd_vel
+              </remapping>
+            </xacro:if>
+            <xacro:unless value="${ros_distro == 'humble'}">
+              <remapping>
+                /diff_drive_controller/cmd_vel:=/cmd_vel
+              </remapping>
+            </xacro:unless>
             <remapping>
               /diff_drive_controller/odom:=/odom

Commit message: mod: update hardware interfaces and controller setup for Jazzy
Signed-off-by: Tomoaki Fujino <fujino.tomoaki404@mail.kyutech.jp>

File: turtlebot3_lime_description/urdf/control/turtlebot3_lime_system.ros2_control.xacro (robot description, xacro)
@@ -13,5 +13,5 @@
       <hardware>
         <xacro:if value="${use_fake_hardware}">
-          <plugin>fake_components/GenericSystem</plugin>
+          <plugin>mock_components/GenericSystem</plugin>
           <param name="fake_sensor_commands">${fake_sensor_commands}</param>
           <param name="state_following_offset">0.0</param>
@@ -33,8 +33,13 @@
         </xacro:unless>
       </hardware>
+      <!--
+        Define the initial command values here to keep the initial commands
+        consistent across hardware, Gazebo, and fake hardware.
+      -->
       <joint name="${prefix}wheel_left_joint">
         <command_interface name="velocity">
           <param name="min">-24.5</param>
           <param name="max">24.5</param>
+          <param name="initial_value">0.0</param>
         </command_interface>
         <state_interface name="position">
@@ -49,4 +54,5 @@
           <param name="min">-24.5</param>
           <param name="max">24.5</param>
+          <param name="initial_value">0.0</param>
         </command_interface>
         <state_interface name="position">
@@ -90,16 +96,15 @@
       </sensor>
       <sensor name="battery">
-        <state_interface name="voltage">
-          <param name="initial_value">0.0</param>
-        </state_interface>
-        <state_interface name="percentage">
-          <param name="initial_value">0.0</param>
-        </state_interface>
-        <state_interface name="design_capacity">
-          <param name="initial_value">0.0</param>
-        </state_interface>
-        <state_interface name="present">
-          <param name="initial_value">0.0</param>
-        </state_interface>
+        <state_interface name="battery_voltage">
+          <param name="initial_value">12.0</param>
+        </state_interface>
+        <state_interface name="battery_percentage">
+          <param name="initial_value">100.0</param>
+        </state_interface>
+        <xacro:unless value="${ros_distro == 'humble'}">
+          <state_interface name="battery_present" data_type="bool">
+            <param name="initial_value">true</param>
+          </state_interface>
+        </xacro:unless>
       </sensor>
       <joint name="${prefix}joint1">
@@ -107,4 +112,5 @@
           <param name="min">${-pi*0.9}</param>
           <param name="max">${pi*0.9}</param>
+          <param name="initial_value">0.0</param>
         </command_interface>
         <state_interface name="position">
@@ -119,19 +125,22 @@
           <param name="min">${-pi*0.57}</param>
           <param name="max">${pi*0.5}</param>
-        </command_interface>
-        <state_interface name="position">
-          <param name="initial_value">0.0</param>
-        </state_interface>
-        <state_interface name="velocity">
-          <param name="initial_value">0.0</param>
-        </state_interface>
-      </joint>
+          <param name="initial_value">-1.10</param>
+        </command_interface>
+        <state_interface name="position">
+          <param name="initial_value">-1.10</param>
+        </state_interface>
+        <state_interface name="velocity">
+          <param name="initial_value">0.0</param>
+        </state_interface>
+      </joint>
+      <!-- FIXME Verify the joint3 limits and set a valid initial position. -->
       <joint name="${prefix}joint3">
         <command_interface name="position">
           <param name="min">${-pi*0.3}</param>
           <param name="max">${pi*0.44}</param>
-        </command_interface>
-        <state_interface name="position">
-          <param name="initial_value">0.0</param>
+          <param name="initial_value">1.80</param>
+        </command_interface>
+        <state_interface name="position">
+          <param name="initial_value">1.80</param>
         </state_interface>
         <state_interface name="velocity">
@@ -143,4 +152,5 @@
           <param name="min">${-pi*0.57}</param>
           <param name="max">${pi*0.65}</param>
+          <param name="initial_value">0.0</param>
         </command_interface>
         <state_interface name="position">
@@ -155,7 +165,8 @@
           <param name="min">${-pi*0.57}</param>
           <param name="max">${pi*0.65}</param>
-        </command_interface>
-        <state_interface name="position">
-          <param name="initial_value">0.0</param>
+          <param name="initial_value">0.98</param>
+        </command_interface>
+        <state_interface name="position">
+          <param name="initial_value">0.98</param>
         </state_interface>
         <state_interface name="velocity">
@@ -167,16 +178,19 @@
           <param name="min">${-pi*0.57}</param>
           <param name="max">${pi*0.65}</param>
-        </command_interface>
-        <state_interface name="position">
-          <param name="initial_value">0.0</param>
-        </state_interface>
-        <state_interface name="velocity">
-          <param name="initial_value">0.0</param>
-        </state_interface>
-      </joint>
+          <param name="initial_value">0.0</param>
+        </command_interface>
+        <state_interface name="position">
+          <param name="initial_value">0.0</param>
+        </state_interface>
+        <state_interface name="velocity">
+          <param name="initial_value">0.0</param>
+        </state_interface>
+      </joint>
+      <!-- FIXME Verify the gripper joint limits against the URDF and teleop commands. -->
       <joint name="${prefix}gripper_left_joint">
         <command_interface name="position">
           <param name="min">-0.010</param>
           <param name="max">0.019</param>
+          <param name="initial_value">0.0</param>
         </command_interface>
         <state_interface name="position">
